File: test/fixtures/benchmark_projects/pass_i2c_sensor_hub/demo.kicad_sch (KiCad schematic)
At the start: 11 parts, among them J1 USB_C, U1 STM32G031G8Ux, U2 BME280, U3 AT24C32, U4 AP2112K-3.3

Commit message: fix(fixtures): spread schematic symbols across A4 sheet via sch_auto_place_functional
Connections:
- net I2C_SCL: no longer U2.3 (SDI)
- net I2C_SDA: no longer U2.4 (SCK)
Other:
- moved on the sheet: C1, C2, C3, C4, J1, R1, R2, U1, U2, U4
